File: ThreeLed/ThreeLedGlobe.kicad_pcb (KiCad board)
At the start: 2 copper layers, 26.8 x 25.5 mm, 9 parts

Commit message: updated
Parts:
- moved   0.67 mm to (164.8, 95.2)
- moved   0.51 mm to (155.2, 95.2)
- moved   0.35 mm to (160.1, 87.5)
- moved   0.07 mm to (154.8, 82.8)
Routing:
- net Net-(LED1-Pad4): track 10.0 -> 11.0 mm
- net Net-(LED2-Pad4): track 13.9 -> 14.7 mm
- net /GND: track 95.2 -> 94.6 mm
Other:
- board text added: "1"
- board text added: "2"
- board text added: "3"
- board text added: "Dodecahedral Light Engine 3 LED V1.2"
- board text added: "V1.2"
- board text removed: "Dodecahedral Light Engine 3 LED V1.1"
- board text removed: "V1.1"

Commit message: updated
Parts:
- added  : , Capacitors_SMD:C_0805, F.Cu at (165.4, 89.8)
Routing:
- net VCC: track 0.00 -> 7.27 mm
- net /GND: track 94.6 -> 90.1 mm
- net GND: track 0.00 -> 3.55 mm
- net Net-(LED1-Pad4): track 11.0 -> 8.17 mm
- net /VCC: track 54.0 -> 52.5 mm
Other:
- board text added: "V1.3"
- board text removed: "V1.2"

Commit message: push
Parts:
- moved   0.31 mm to (164.5, 95.2)
- moved   0.30 mm to (155.4, 95.2)
Routing:
- net /DOUT: track 71.4 -> 73.3 mm
- net /DIN: track 71.5 -> 69.7 mm
- net /GND: track 90.1 -> 91.8 mm, vias 1 -> 0
Other:
- board text added: "Dodecahedral Light Engine 3 LED V1.3"
- board text removed: "Dodecahedral Light Engine 3 LED V1.2"
